File: hardware/rook/rook.kicad_sch (KiCad schematic)
At the start: 29 parts, among them J1 Conn_01x02_Socket, J10 Micro_SD_Card, J2 Conn_01x04_Pin, J3 Conn_01x04_Pin, J4 Conn_01x01_Socket, J6 Conn_01x04_Socket, J7 Screw_Terminal_01x03, J8 Conn_01x03_Socket, J9 Conn_01x10_Socket, SW1 SW_Push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

Commit message: update
Connections:
- net A0: no longer SW1.1, U2.18 (AIN0/P0.02)
- net A5_SD: no longer J10.2 (DAT3/CD), SW2.1, U2.19 (AIN5/P0.29)
- net BUSY: now also U2.19 (AIN5/P0.29); no longer U2.8 (P0.24)
- net MISO: now also U2.18 (AIN0/P0.02); no longer U2.9 (P1.00)
- net P1_06: now also J10.2 (DAT3/CD)
- new net BUTTON_A: SW1.1, U2.9 (P1.00)
- new net BUTTON_B: SW2.1, U2.8 (P0.24)

Commit message: update
Parts:
- added JP1, JP2, JP3: Jumper_2_Open, Jumper:SolderJumper-2_P1.3mm_Open_Pad1.0x1.5mm, symbol Jumper:Jumper_2_Open
- added Q2: 2N7002, Package_TO_SOT_SMD:SOT-23, symbol Transistor_FET:2N7002
- added R12, R13, R14, R15, R18: R, Resistor_SMD:R_0805_2012Metric_Pad1.20x1.40mm_HandSolder, symbol Device:R
- added R16: 10K, Resistor_SMD:R_0805_2012Metric_Pad1.20x1.40mm_HandSolder, symbol Device:R
- added U3: PCF8574, Package_SO:SOIC-16W_7.5x10.3mm_P1.27mm, symbol Interface_Expansion:PCF8574
Connections:
- net 3V3: now also U3.13 (~{INT}), U3.16 (VDD)
- net BUTTON_B: now also U3.4 (P0); no longer U2.8 (P0.24)
- net GND: now also JP3.1 (A), Q2.2 (S), R12.1, R13.1, R14.1, R16.1, U3.8 (VSS); no longer J2.4 (Pin_4)
- net GPS_RX: now also JP2.2 (B), R15.2; no longer J2.2 (Pin_2)
- net GPS_TX: now also JP1.2 (B), R18.2; no longer J2.3 (Pin_3)
- net P1_06: no longer SW3.1
- net SCL: now also U3.14 (SCL)
- net SDA: now also U3.15 (SDA)
- net A0 renamed P2
- net P2: now also U3.6 (P2)
- net A5_SD renamed P3
- net P3: now also U3.7 (P3)
- net CS renamed LORA_CS
- new net: R13.2, U3.2 (A1)
- new net: J2.2 (Pin_2), JP2.1 (A), R15.1
- new net: R14.2, U3.1 (A0)
- new net: R12.2, U3.3 (A2)
- new net: J2.3 (Pin_3), JP1.1 (A), R18.1
- new net BUTTON_C: SW3.1, U3.5 (P1)
- new net GPS_EN: Q2.1 (G), R16.2, U2.8 (P0.24)
- new net GPS_GND: J2.4 (Pin_4), JP3.2 (B), Q2.3 (D)
- new net P4: U3.9 (P4)
- new net P5: U3.10 (P5)
- new net P6: U3.11 (P6)
- new net P7: U3.12 (P7)
Other:
- note added: "Display"
- note added: "Mesh GPS"
- note added: "Qwiic"
- note removed: "Meshtastic Display"
- note removed: "Meshtastic GPS"
- moved on the sheet: J1, J10, J2, J3, J4, J6, J7, J8, R1, R10, R2, R5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
