File: hardware/rook/rook.kicad_pcb (KiCad board)
At the start: 2 copper layers, 77.9 x 50 mm, 29 parts, among them J1 Conn_01x02_Socket, J10 Micro_SD_Card, J2 Conn_01x04_Pin, J3 Conn_01x04_Pin, J4 Conn_01x01_Socket, J6 Conn_01x04_Socket, J7 Screw_Terminal_01x03, J8 Conn_01x03_Socket, J9 Conn_01x10_Socket, SW1 SW_Push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

Commit message: update
Parts:
- moved SW1 107.4 mm to (71.5, 6.30)
- moved SW2 107.0 mm to (71.5, 16.0)
- moved SW3 107.0 mm to (71.5, 25.9)
- moved J8 106.8 mm to (72.6, 38.3)
- moved J2 106.6 mm to (47.2, 35.1)
- moved H3 106.6 mm to (72.0, 0.00)
- moved SW4 106.5 mm to (4.30, 5.60)
- moved J9 106.4 mm to (42.2, 41.9)
- moved J6 106.3 mm to (36.5, 42.5)
- moved J10 106.3 mm to (12.9, 1.95)
- moved U4 106.2 mm to (13.3, 41.5)
- moved J1 106.1 mm to (1.75, 36.8)
- moved J3 106.1 mm to (54.5, -0.44)
- moved J4 106.1 mm to (28.2, -1.04)
- moved R4 106.1 mm to (57.7, 12.0)
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Other:
- board size 77.9 x 50 mm -> 79 x 51 mm
- board text added: "P0_20"
- board text added: "P0_22"
- board text added: "P1_06"
- board text added: "Qwiic"
- board text added: "RX"
- board text added: "TX"
- board text removed: "GPS_RX"
- board text removed: "GPS_TX"
- board text removed: "Qwiic/ Stemma QT"

Commit message: update
Parts:
- moved SW1 0.49 mm to (72.0, 6.25)
- moved SW2 0.49 mm to (72.0, 15.9)
- moved SW3 0.49 mm to (72.0, 25.8)
Connections:
- J10 pad 2: A5_SD -> P1_06
- SW1 pad 1: A0 -> BUTTON_A
- SW2 pad 1: A5_SD -> BUTTON_B
- U2 pad 18: A0 -> MISO
- U2 pad 19: A5_SD -> BUSY
- U2 pad 8: BUSY -> BUTTON_B
- U2 pad 9: MISO -> BUTTON_A
Other:
- board text added: "A"
- board text added: "B"
- board text added: "C"
Changed lines of the file:
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@@
 	(net 26 "unconnected-(J10-DAT2-Pad1)")
 	(net 27 "unconnected-(J10-DAT1-Pad8)")
+	(net 28 "BUTTON_A")
+	(net 29 "BUTTON_B")
 	(footprint "footprints:JST_SH4_SKINNY"
 		(layer "F.Cu")
@@
 			(layers "*.Cu" "*.SilkS" "*.Mask")
 			(remove_unused_layers no)
-			(net 13 "BUSY")
+			(net 29 "BUTTON_B")
 			(pinfunction "P0.24")
 			(pintype "input")
@@
 			(layers "*.Cu" "*.SilkS" "*.Mask")
 			(remove_unused_layers no)
-			(net 16 "MISO")
+			(net 28 "BUTTON_A")
 			(pinfunction "P1.00")
 			(pintype "input")
@@
 			(layers "*.Cu" "*.SilkS" "*.Mask")
 			(remove_unused_layers no)
-			(net 11 "A0")
+			(net 16 "MISO")
 			(pinfunction "AIN0/P0.02")
 			(pintype "input")
@@
 			(layers "*.Cu" "*.SilkS" "*.Mask")
 			(remove_unused_layers no)
-			(net 2 "A5_SD")
+			(net 13 "BUSY")
 			(pinfunction "AIN5/P0.29")
 			(pintype "input")
@@
 	(footprint "Button_Switch_THT:SW_Tactile_SPST_Angled_PTS645Vx31-2LFS"
 		(layer "F.Cu")
-		(at 71.5 6.3 -90)
+		(at 71.99 6.25 -90)
 		(descr "tactile switch SPST right angle, PTS645VL31-2 LFS")
 		(tags "tactile switch SPST angled PTS645VL31-2 LFS C&K Button")
@@
 			(at 2.3 2.25 90)
 			(layer "F.SilkS")
+			(hide yes)
 			(effects
 				(font
@@
 			(layers "*.Cu" "*.Mask")
 			(remove_unused_layers no)
-			(net 11 "A0")
+			(net 28 "BUTTON_A")
 			(pinfunction "1")
 			(pintype "passive")
@@
 			(size 0.7 1.75)
 			(layers "F.Cu" "F.Paste" "F.Mask")
-			(net 2 "A5_SD")
+			(net 1 "P1_06")
 			(pinfunction "DAT3/CD")
 			(pintype "bidirectional")
@@
 	(footprint "Button_Switch_THT:SW_Tactile_SPST_Angled_PTS645Vx31-2LFS"
 		(layer "F.Cu")
-		(at 71.5 16 -90)
+		(at 71.99 15.95 -90)
 		(descr "tactile switch SPST right angle, PTS645VL31-2 LFS")
 		(tags "tactile switch SPST angled PTS645VL31-2 LFS C&K Button")
@@
 			(at 2.45 2.25 90)
 			(layer "F.SilkS")
+			(hide yes)
 			(effects
 				(font
@@
 			(layers "*.Cu" "*.Mask")
 			(remove_unused_layers no)
-			(net 2 "A5_SD")
+			(net 29 "BUTTON_B")
 			(pinfunction "1")
 			(pintype "passive")
@@
 	(footprint "Button_Switch_THT:SW_Tactile_SPST_Angled_PTS645Vx31-2LFS"
 		(layer "F.Cu")
-		(at 71.5 25.85 -90)
+		(at 71.99 25.8 -90)
 		(descr "tactile switch SPST right angle, PTS645VL31-2 LFS")
 		(tags "tactile switch SPST angled PTS645VL31-2 LFS C&K Button")
@@
 			(at 2.39 2.25 90)
 			(layer "F.SilkS")
+			(hide yes)
 			(effects
 				(font
@@
 		)
 	)
+	(gr_text "B"
+		(at 68.39 19.05 0)
+		(layer "F.SilkS")
+		(effects
+			(font
+				(size 1.5 1.5)
+				(thickness 0.3)
+				(bold yes)
+			)
+			(justify left bottom)
+		)
+	)
 	(gr_text "RST"
 		(at -1.55 10.15 90)
@@
 		)
 	)
+	(gr_text "C"
+		(at 68.34 29 0)
+		(layer "F.SilkS")
+		(effects
+			(font
+				(size 1.5 1.5)
+				(thickness 0.3)
+				(bold yes)
+			)
+			(justify left bottom)
+		)
+	)
 	(gr_text "v0.1"
 		(at 58.65 35.685 0)
@@
 			)
 			(justify left bottom)
+		)
+	)
+	(gr_text "A"
+		(at 68.19 9.55 0)
+		(layer "F.SilkS")
+		(effects
+			(font
+				(size 1.5 1.5)
+				(thickness 0.3)
+				(bold yes)
+			)
+			(justify left bottom)

Commit message: update
Parts:
- added JP1: Jumper_2_Open, Jumper:SolderJumper-2_P1.3mm_Open_Pad1.0x1.5mm, F.Cu at (59.3, 22.1)
- added JP2: Jumper_2_Open, Jumper:SolderJumper-2_P1.3mm_Open_Pad1.0x1.5mm, F.Cu at (53.7, 22.2)
- added JP3: Jumper_2_Open, Jumper:SolderJumper-2_P1.3mm_Open_Pad1.0x1.5mm, F.Cu at (38.0, 18.6)
- added Q2: 2N7002, Package_TO_SOT_SMD:SOT-23, F.Cu at (41.8, 19.7)
- added R12: R, Resistor_SMD:R_0805_2012Metric_Pad1.20x1.40mm_HandSolder, F.Cu at (44.8, 13.2)
- added R13: R, Resistor_SMD:R_0805_2012Metric_Pad1.20x1.40mm_HandSolder, F.Cu at (44.8, 10.8)
- added R14: R, Resistor_SMD:R_0805_2012Metric_Pad1.20x1.40mm_HandSolder, F.Cu at (44.9, 8.75)
- added R15: R, Resistor_SMD:R_0805_2012Metric_Pad1.20x1.40mm_HandSolder, F.Cu at (49.7, 22.2)
- added R16: 10K, Resistor_SMD:R_0805_2012Metric_Pad1.20x1.40mm_HandSolder, F.Cu at (46.0, 18.0)
- added R18: R, Resistor_SMD:R_0805_2012Metric_Pad1.20x1.40mm_HandSolder, F.Cu at (61.6, 22.1)
- added U3: PCF8574, Package_SO:SOIC-16W_7.5x10.3mm_P1.27mm, F.Cu at (55.4, 12.0)
- moved U4 52.4 mm to (65.7, 42.0)
- moved J9 35.9 mm to (6.40, 42.1)
- moved J6 16.0 mm to (52.5, 42.8)
- moved J7 15.5 mm to (34.5, 40.1)
- moved R4 13.8 mm to (63.8, -0.45)
- moved R8 13.8 mm to (61.3, -0.40)
- moved R7 13.7 mm to (40.1, -0.55)
- moved R3 13.7 mm to (42.5, -0.60)
- moved J2 3.02 mm to (50.2, 35.5)
- moved SW2 2.40 mm to (72.0, 18.4)
- moved SW3 2.35 mm to (72.0, 28.1)
- moved J8 1.34 mm to (71.4, 38.9)
- moved R6 0.75 mm to (13.3, 23.9)
- moved R1 0.75 mm to (13.3, 26.5)
- moved R2 0.75 mm to (7.15, 21.5)
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Connections:
- net CS renamed LORA_CS
- J2 pad 2: GPS_RX -> Net-(J2-Pin_2)
- J2 pad 3: GPS_TX -> Net-(J2-Pin_3)
- J2 pad 4: GND -> GPS_GND
- J9 pad 10: A5_SD -> P3
- J9 pad 9: A0 -> P2
- SW3 pad 1: P1_06 -> BUTTON_C
- U2 pad 8: BUTTON_B -> GPS_EN
Other:
- board text added: "GPS_GND"
- board text added: "P2"
- board text added: "P3"
- board text added: "rook"
- board text removed: "A0"
- board text removed: "A5"

Commit message: update
Parts:
- moved R16 6.20 mm to (48.0, 23.9)
- moved JP3 5.17 mm to (39.3, 23.6)
- moved Q2 4.32 mm to (43.6, 23.6)
- moved R18 2.65 mm to (63.6, 23.9)
- moved JP2 2.44 mm to (55.5, 23.9)
- moved R15 2.44 mm to (51.5, 23.9)
- moved J1 2.31 mm to (4.20, 37.4)
- moved JP1 1.82 mm to (59.8, 23.9)
- moved SW2 1.05 mm to (72.0, 17.3)
- moved R12 0.63 mm to (45.0, 13.8)
- moved R13 0.56 mm to (44.8, 11.3)
- moved R14 0.22 mm to (44.8, 8.95)
- moved R8 0.20 mm to (61.3, -0.60), turned to 180 degrees
- moved R4 0.13 mm to (63.8, -0.57)
- moved R3 0.09 mm to (42.6, -0.58)
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Routing:
- net GND: track 0.00 -> 326.6 mm, vias 0 -> 36
- net 3V3: track 0.00 -> 239.6 mm, vias 0 -> 24
- net SCL: track 0.00 -> 139.4 mm, vias 0 -> 10
- net BAT: track 0.00 -> 130.5 mm, vias 0 -> 9
- net SDA: track 0.00 -> 124.7 mm, vias 0 -> 11
- net V_EXT: track 0.00 -> 79.1 mm, vias 0 -> 4
- net BUTTON_A: track 0.00 -> 73.7 mm, vias 0 -> 3
- net P1_06: track 0.00 -> 66.7 mm, vias 0 -> 4
- net GPS_TX: track 0.00 -> 54.4 mm, vias 0 -> 4
- net GPS_RX: track 0.00 -> 53.5 mm, vias 0 -> 4
- net P2: track 0.00 -> 51.0 mm, vias 0 -> 4
- net P3: track 0.00 -> 46.2 mm, vias 0 -> 4
- net BUTTON_C: track 0.00 -> 36.8 mm, vias 0 -> 3
- net GPS_EN: track 0.00 -> 35.3 mm, vias 0 -> 3
- net GPS_GND: track 0.00 -> 31.7 mm, vias 0 -> 4
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Other:
- board text added: "design files and code:"
