File: hardware/v0.2/rook/rook.kicad_pcb (KiCad board)
At the start: 2 copper layers, 91.2 x 53.1 mm, 41 parts, among them J1 Conn_01x02_Socket, J10 Micro_SD_Card, J11 Conn_01x04_Pin, J2 Conn_01x04_Pin, J3 Conn_01x04_Pin, J4 Conn_01x01_Socket, J6 Conn_01x04_Socket, J7 Screw_Terminal_01x03, J8 Conn_01x03_Socket, J9 Conn_01x10_Socket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

Commit message: update
Parts:
- moved J6 25.4 mm to (19.7, 118.4)
- moved J10 19.7 mm to (53.5, 118.8)
- moved J7 16.4 mm to (29.7, 116.1)
- moved TFT_BL1 12.2 mm to (65.7, 107.5), turned to 0 degrees
- moved J1 4.51 mm to (-17.2, 91.6)
- moved U4 2.75 mm to (9.50, 117.5)
- moved RESET1 1.41 mm to (-3.65, 120.5)
- moved U1 0.53 mm to (19.3, 82.6)
- moved H1 0.52 mm to (-16.9, 120.3)
- moved H4 0.28 mm to (-16.8, 73.6)
- moved J8 0.20 mm to (-15.2, 113.1)
