File: hardware/v0.3/rook/rook.kicad_sch (KiCad schematic)
At the start: 41 parts, among them J1 Conn_01x02_Socket, J10 Micro_SD_Card, J11 Conn_01x04_Pin, J2 Conn_01x04_Pin, J3 Conn_01x04_Pin, J4 Conn_01x01_Socket, J6 Conn_01x04_Socket, J7 Screw_Terminal_01x03, J8 Conn_01x03_Socket, J9 Conn_01x10_Socket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

Commit message: update
Parts:
- removed J9: Conn_01x10_Socket, Connector_PinSocket_2.54mm:PinSocket_1x10_P2.54mm_Vertical, symbol Connector:Conn_01x10_Socket
- removed U3: ~, footprints:st7789_tft_2in_320x240, symbol lucc:st7789
- added R11, R12, R13, R14, R19, R21, R23: R, Resistor_THT:R_Axial_DIN0207_L6.3mm_D2.5mm_P10.16mm_Horizontal, symbol Device:R
- added R17, R20, R22, R24: R, Resistor_SMD:R_0805_2012Metric_Pad1.20x1.40mm_HandSolder, symbol Device:R
- J8, TFT_BL1: footprint footprints:usual_switch -> eg1206:SSW_1825232-1
- R1, R10, R2, R3, R4: footprint Resistor_THT:R_Axial_DIN0204_L3.6mm_D1.6mm_P5.08mm_Horizontal -> Resistor_THT:R_Axial_DIN0207_L6.3mm_D2.5mm_P10.16mm_Horizontal
- U1: footprint wio-sx1262:wio-sx1262 -> wio-sx1262:wio-sx1262-extended
Connections:
- net 3V3: now also U5.7 (VCC), R14.2, R17.2, R19.2, R20.2, R21.2, R22.2, R23.2, R24.2; no longer U5.1 (VCC)
- net BUTTON_A: now also R19.1, R20.1
- net GND: now also U5.8 (GND), R13.2; no longer U5.1 (VCC)
- net GPS_EN: now also R13.1
- net GPS_RX: now also R12.2
- net GPS_TX: now also R11.2
- net MESH_RST: now also U5.4 (RST), R14.1, R17.1; no longer U5.1 (VCC)
- net MOSI: now also U5.5 (MOSI); no longer U5.1 (VCC)
- net P0_6: now also U5.3 (DC), R21.1, R22.1; no longer U5.1 (VCC)
- net P0_8: now also U5.2 (CS), R23.1, R24.1; no longer U5.1 (VCC)
- net SCK: now also U5.6 (SCK); no longer U5.1 (VCC)
- net at J2.2 (Pin_2), JP2.1 (A), R15.1: now also R12.1
- net at J2.3 (Pin_3), JP1.1 (A), R18.1: now also R11.1
Other:
- note removed: "Breakouts"
- note removed: "ST7789 TFT 2 IN"
- moved on the sheet: B1, B2, B3, J2, J8, JP1, JP2, JP3, Q2, R15, R16, R18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
