File: hardware/v0.4/rook/rook.kicad_pcb (KiCad board)
At the start: 2 copper layers, 79.3 x 46.4 mm, 50 parts, among them J1 Conn_01x02_Socket, J10 Micro_SD_Card, J11 Conn_01x04_Pin, J2 Conn_01x04_Pin, J3 Conn_01x04_Pin, J4 Conn_01x01_Socket, J6 Conn_01x04_Socket, J7 Screw_Terminal_01x03, J8 Conn_01x03_Socket, Q2 2N7002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

Commit message: new layout
Parts:
- added J5: Conn_01x04_Socket, Connector_PinSocket_2.54mm:PinSocket_1x04_P2.54mm_Vertical, F.Cu at (20.2, 33.8)
- J8, TFT_BL1: footprint eg1206:SSW_1825232-1 -> footprints:SSW_1825232-1
- moved J1 2.27 mm to (25.7, 41.0)
- moved U4 1.44 mm to (38.3, 36.9)
- moved J7 0.86 mm to (43.8, 36.3)
- moved J8 0.80 mm to (13.3, 40.5)
- moved TFT_BL1 0.79 mm to (65.8, 40.4)
- moved U2 0.33 mm to (16.1, 22.7)
- moved R7 0.25 mm to (39.3, 19.1)
- moved R10 0.20 mm to (46.0, 24.8)
- moved U5 0.20 mm to (58.9, 0.60)
- moved R9 0.20 mm to (46.0, 19.1)
- moved R12 0.18 mm to (49.4, 14.6)
- moved R11 0.17 mm to (52.7, 14.6)
- moved R13 0.15 mm to (56.0, 14.6)
- moved R15 0.15 mm to (49.4, 19.1)
- moved R16 0.12 mm to (56.0, 19.1)
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Routing:
- net GND: track 309.6 -> 0.00 mm, vias 30 -> 0
- net 3V3: track 224.9 -> 0.00 mm, vias 20 -> 0
- net P0_6: track 114.9 -> 0.00 mm, vias 6 -> 0
- net P0_8: track 101.9 -> 0.00 mm, vias 3 -> 0
- net P1_06: track 91.2 -> 0.00 mm, vias 6 -> 0
- net SCL: track 88.7 -> 0.00 mm, vias 13 -> 0
- net MESH_RST: track 82.9 -> 0.00 mm, vias 8 -> 0
- net SDA: track 81.9 -> 0.00 mm, vias 8 -> 0
- net BUTTON_A: track 78.7 -> 0.00 mm, vias 3 -> 0
- net MOSI: track 68.2 -> 0.00 mm, vias 6 -> 0
- net GPS_RX: track 66.4 -> 0.00 mm, vias 6 -> 0
- net GPS_EN: track 63.9 -> 0.00 mm, vias 4 -> 0
- net GPS_TX: track 60.9 -> 0.00 mm, vias 3 -> 0
- net SCK: track 56.1 -> 0.00 mm, vias 7 -> 0
- net BAT: track 52.2 -> 0.00 mm, vias 4 -> 0
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Other:
- board text added: "D0"
- board text added: "D1"
- board text added: "v0.4"
- board text removed: "P0.6"
- board text removed: "P0.8"
- board text removed: "v0.3"
