File: hardware/v0.4/rook/rook.kicad_pcb (KiCad board)
At the start: 2 copper layers, 79.3 x 46.4 mm, 51 parts, among them J1 Conn_01x02_Socket, J10 Micro_SD_Card, J11 Conn_01x04_Pin, J2 Conn_01x04_Pin, J3 Conn_01x04_Pin, J4 Conn_01x01_Socket, J5 Conn_01x04_Socket, J6 Conn_01x04_Socket, J7 Screw_Terminal_01x03, J8 Conn_01x03_Socket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

Commit message: tweaks
Parts:
- moved R19 1.59 mm to (18.0, 24.4)
- moved R20 1.55 mm to (22.4, 24.4)
- moved R6 1.54 mm to (8.53, 18.9)
- moved R1 1.54 mm to (14.1, 18.9)
- moved R2 1.54 mm to (4.03, 24.4)
- moved R5 1.54 mm to (8.65, 24.3)
- moved R14 1.54 mm to (18.0, 18.9)
- moved R17 1.54 mm to (22.5, 18.9)
Routing:
- net 3V3: track 0.00 -> 240.0 mm, vias 0 -> 26
- net GND: track 0.00 -> 223.8 mm, vias 0 -> 26
- net BAT: track 0.00 -> 52.6 mm, vias 0 -> 4

Commit message: update
Routing:
- net P0_8: track 0.00 -> 125.8 mm, vias 0 -> 8
- net P0_6: track 0.00 -> 122.9 mm, vias 0 -> 7
- net SCL: track 0.00 -> 99.1 mm, vias 0 -> 11
- net BUTTON_A: track 0.00 -> 88.3 mm, vias 0 -> 8
- net P1_06: track 0.00 -> 87.9 mm, vias 0 -> 6
- net MESH_RST: track 0.00 -> 84.2 mm, vias 0 -> 8
- net SDA: track 0.00 -> 82.8 mm, vias 0 -> 10
- net GPS_RX: track 0.00 -> 67.6 mm, vias 0 -> 4
- net GPS_TX: track 0.00 -> 65.5 mm, vias 0 -> 5
- net GPS_EN: track 0.00 -> 64.6 mm, vias 0 -> 7
- net SCK: track 0.00 -> 60.3 mm, vias 0 -> 6
- net MOSI: track 0.00 -> 58.0 mm, vias 0 -> 9
- net Net-(J2-Pin_3): track 0.00 -> 49.9 mm, vias 0 -> 6
- net RF_SW: track 0.00 -> 45.6 mm, vias 0 -> 3
- net Backlight: track 0.00 -> 45.6 mm, vias 0 -> 1
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
Commit message: finished routing
Routing:
- net GND: track 262.1 -> 281.0 mm, vias 30 -> 32
- net 3V3: track 245.3 -> 257.0 mm, vias 28 -> 27
- net GPS_TX: track 65.5 -> 64.4 mm
- net P1_06: track 87.9 -> 88.6 mm
Other:
- board text added: "1-wire"
- board text added: "GROVE"
- board text added: "microSD"
- board text added: "wio-SX1262"
- board text removed: "1W"
